File: breadboard_power_supply/breadboard_power_supply.kicad_pcb (KiCad board)
At the start: 2 copper layers, 34.2 x 58.5 mm, 17 parts, among them J1 Conn_01x02_Pin, J2 Conn_01x02_Pin, J3 Conn_01x03_Pin, J4 Conn_01x03_Pin, J5 Screw_Terminal_01x02, J6 Barrel_Jack_PTH, J7 Screw_Terminal_01x02, U2 LM317_TO-220, U3 LM7805_TO220

Commit message: final DRC fixes
Routing:
- net /12V: track 58.4 -> 61.0 mm
- net /5V: track 68.2 -> 70.4 mm
- net Net-(U2-ADJ): track 46.3 -> 47.8 mm
Other:
- board text added: "+"
- board text added: "-"
- board text added: "3.3V"
- board text added: "5V"
- board text added: "GND"
- board text added: "Jose Padilla * 2025"
- board text added: "OFF"
- board text added: "ON"
- board text added: "v1"

Commit message: final design DRC fixes
Connections:
- J1 pad 2: /PWR_OUTPUT -> /POWER_OUT_TOP
- J2 pad 2: /PWR_OUTPUT -> /POWER_OUT_BOTTOM
- J3 pad 2: /PWR_OUTPUT -> /POWER_OUT_BOTTOM
- J4 pad 2: /PWR_OUTPUT -> /POWER_OUT_TOP
- J5 pad 2: /PWR_OUTPUT -> /POWER_OUT_TOP
- J7 pad 2: /PWR_OUTPUT -> /POWER_OUT_BOTTOM
Routing:
- net /PWR_OUTPUT: track 86.7 -> 0.00 mm
- net /POWER_OUT_BOTTOM: track 0.00 -> 20.2 mm
- net /POWER_OUT_TOP: track 0.00 -> 19.6 mm
