File: breadboard_power_supply/breadboard_power_supply.kicad_sch (KiCad schematic)
At the start: 17 parts, among them J1 Conn_01x02_Pin, J2 Conn_01x02_Pin, J3 Conn_01x03_Pin, J4 Conn_01x03_Pin, J5 Screw_Terminal_01x02, J6 Barrel_Jack_PTH, J7 Screw_Terminal_01x02, U2 LM317_TO-220, U3 LM7805_TO220

Commit message: final design DRC fixes
Connections:
- net PWR_OUTPUT renamed POWER_OUT_BOTTOM
- net POWER_OUT_BOTTOM: no longer J1.2 (Pin_2), J4.2 (Pin_2), J5.2 (Pin_2)
- new net POWER_OUT_TOP: J1.2 (Pin_2), J4.2 (Pin_2), J5.2 (Pin_2)
