File: mcu_datalogger/mcu_datalogger.kicad_pcb (KiCad board)
At the start: 2 copper layers, 51.9 x 31.1 mm, 29 parts, among them J1 Conn_01x04_Pin, J2 Conn_01x04_Pin, J3 Conn_01x09, J4 Conn_02x03_Odd_Even, U1 24LC1025, U2 24LC1025, U3 DS1337S_, U4 ATMEGA328P-AU, Y1 16 MHz, Y2 32.768KHz

Commit message: back copper
Routing:
- added copper zone on B.Cu, net GND
Changed lines of the file:
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@@
 		(net 26)
+	)
+	(zone
+		(net 2)
+		(net_name "GND")
+		(layer "B.Cu")
+		(name "back copper")
+		(hatch edge 0.5)
+		(connect_pads
+			(clearance 0.5)
+		)
+		(min_thickness 0.25)
+		(filled_areas_thickness no)
+		(fill yes
+			(thermal_gap 0.5)
+			(thermal_bridge_width 0.5)
+		)
+		(polygon
+			(pts
+				(xy 114.808 44.577) (xy 114.808 75.311) (xy 62.992 75.311) (xy 62.992 44.577)
+			)
+		)
 	)
 	(embedded_fonts no)

Commit message: back silkscreen details
Other:
- board text added: "${project_name} v1 Jose Padilla 2025"
Changed lines of the file:
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@@
 		(layer "Edge.Cuts")
+	)
+	(gr_text "${project_name}\nv1\nJose Padilla\n2025\n"
+		(at 82.9 52 0)
+		(layer "B.SilkS")
+		(effects
+			(font
+				(size 1 1)
+				(thickness 0.1)
+			)
+			(justify left bottom mirror)
+		)
 	)
 	(segment

Commit message: back copper vias
Routing:
- net GND: track 174.2 -> 175.1 mm
- net Net-(D1-K): track 10.1 -> 10.7 mm
