File: mcu_datalogger/mcu_datalogger.kicad_pcb (KiCad board)
At the start: 2 copper layers, 51.9 x 31.1 mm, 29 parts, among them J1 Conn_01x04_Pin, J2 Conn_01x04_Pin, J3 Conn_01x09, J4 Conn_02x03_Odd_Even, U1 24LC1025, U2 24LC1025, U3 DS1337S_, U4 ATMEGA328P-AU, Y1 16 MHz, Y2 32.768KHz

Commit message: fix design error
Parts:
- Y1: value 16 MHz -> 16MHz
- Y2: value 32.768KHz -> 32.768 KHz
- moved R5 35.4 mm to (70.2, 61.0)
- moved D2 7.65 mm to (103.8, 52.1)
- moved R4 6.72 mm to (97.5, 52.1)
- moved U1 3.18 mm to (88.9, 48.3)
- moved U2 2.76 mm to (77.5, 48.3)
- moved Y2 2.01 mm to (69.8, 55.2)
- moved Y1 1.91 mm to (71.1, 66.0)
Connections:
- J1 pad 4: /SCK -> /SCL
- R5 pad 2: /SCK -> /SCL
- U1 pad 6: /SCK -> /SCL
- U2 pad 6: /SCK -> /SCL
- U3 pad 6: /SCK -> /SCL
- U4 pad 28: /SCK -> /SCL
Routing:
- net GND: track 175.1 -> 41.6 mm, vias 2 -> 15
- net /SCK: track 108.1 -> 23.6 mm, vias 4 -> 0
- net /SCL: track 0.00 -> 53.6 mm
- net /SDA: track 84.4 -> 51.3 mm, vias 2 -> 3
- net /TX: track 28.9 -> 21.9 mm
- net VCC: track 40.7 -> 33.9 mm, vias 1 -> 0
- net /D3: track 20.4 -> 26.1 mm
- net /RESET: track 30.1 -> 25.3 mm
- net Net-(U3-SQW/~INT): track 22.6 -> 18.4 mm
- net /D6: track 20.4 -> 16.5 mm, vias 1 -> 0
- net Net-(U4-AREF): track 18.1 -> 14.5 mm
- net /D7: track 16.3 -> 19.7 mm, vias 0 -> 1
- net /RX: track 29.5 -> 26.6 mm
- net /Vcc: track 179.1 -> 181.8 mm, vias 4 -> 0
- net /MOSI: track 26.6 -> 29.0 mm
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