File: esp32_iot_manager/user_interface.kicad_sch (KiCad schematic)
At the start: 0 parts

Commit message: sensor and user interface done
Parts:
- added C12, C21: 0.1u, Capacitor_SMD:C_0805_2012Metric, symbol PCM_SL_Devices:Capacitor_NP
- added J4: Conn_01x04_Pin, Connector_PinHeader_2.54mm:PinHeader_1x04_P2.54mm_Vertical, symbol Connector:Conn_01x04_Pin
- added J5: Conn_01x05_Pin, Connector_PinHeader_2.54mm:PinHeader_1x04_P2.54mm_Vertical, symbol Connector:Conn_01x05_Pin
- added Q2, Q3: BC817, Package_TO_SOT_SMD:SOT-23, symbol Transistor_BJT:BC817
- added R32, R33, R34: 10K, Resistor_SMD:R_0805_2012Metric, symbol PCM_SL_Resistors:Resistor
- added S1, S2: USLPT2819DT2TR, USLPT2819DT2TR:SW_USLPT2819DT2TR, symbol USLPT2819DT2TR:USLPT2819DT2TR
Connections:
- new net: Q3.1 (B), R34.2
- new net: Q2.1 (B), R33.2
- new net 3.3V: J4.1 (Pin_1), J5.1 (Pin_1), R32.2
- new net BOOT: C21.1, Q3.2 (E), S1.3, S1.4
- new net DTR: Q3.3 (C), R33.1
- new net EN: C12.1, Q2.3 (C), R32.1, S2.3, S2.4
- new net GND: C12.2, C21.2, J4.4 (Pin_4), J5.5 (Pin_5), S1.1, S1.2, S2.1, S2.2
- new net GPIO18: J5.3 (Pin_3)
- new net GPIO19: J5.4 (Pin_4)
- new net GPIO8: J5.2 (Pin_2)
- new net RTS: Q2.2 (E), R34.1
- new net SCL: J4.3 (Pin_3)
- new net SDA: J4.2 (Pin_2)
Other:
- note added: "Boot"
- note added: "Breakout pins"
- note added: "OLED display connector (12C)"
- note added: "Reset"
- note added: "Reset/boot buttons"
- title: (none) -> User interface

Commit message: finished design of pcb, next copper zones, routing
Parts:
- J5: footprint Connector_PinHeader_2.54mm:PinHeader_1x04_P2.54mm_Vertical -> Connector_PinHeader_2.54mm:PinHeader_1x05_P2.54mm_Vertical
- S1, S2: footprint USLPT2819DT2TR:SW_USLPT2819DT2TR -> esp32_manager_project:SW_USLPT2819DT2TR
Changed lines of the file:
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@@
 			)
 		)
-		(property "Footprint" "Connector_PinHeader_2.54mm:PinHeader_1x04_P2.54mm_Vertical"
+		(property "Footprint" "Connector_PinHeader_2.54mm:PinHeader_1x05_P2.54mm_Vertical"
 			(at 31.75 57.15 0)
 			(effects
@@
 			)
 		)
-		(property "Footprint" "USLPT2819DT2TR:SW_USLPT2819DT2TR"
+		(property "Footprint" "esp32_manager_project:SW_USLPT2819DT2TR"
 			(at 71.12 102.87 0)
 			(effects
@@
 			)
 		)
-		(property "Footprint" "USLPT2819DT2TR:SW_USLPT2819DT2TR"
+		(property "Footprint" "esp32_manager_project:SW_USLPT2819DT2TR"
 			(at 30.48 102.87 0)
 			(effects

Commit message: flip transistor
Connections:
- net BOOT: now also Q3.3 (C); no longer Q3.2 (E)
- net DTR: now also Q3.2 (E); no longer Q3.3 (C)
Changed lines of the file:
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@@
 		(lib_id "Transistor_BJT:BC817")
 		(at 43.18 147.32 0)
+		(mirror x)
 		(unit 1)
 		(exclude_from_sim no)
@@
 		(on_board yes)
 		(dnp no)
-		(fields_autoplaced yes)
 		(property "Reference" "Q3"
-			(at 48.26 146.0499 0)
+			(at 48.26 148.5901 0)
 			(effects
 				(font
@@
 		)
 		(property "Value" "BC817"
-			(at 48.26 148.5899 0)
+			(at 48.26 146.0501 0)
 			(effects
 				(font
@@
 		)
 		(property "Footprint" "Package_TO_SOT_SMD:SOT-23"
-			(at 48.26 149.225 0)
+			(at 48.26 145.415 0)
 			(effects
 				(font
