File: esp32_iot_manager/esp32_iot_manager.kicad_sch (KiCad schematic)
At the start: 0 parts

Commit message: Created symbols, footprints, configs Voltage regulator Next esp32 section, memory, sd card
Parts:
- added C1, C2, C4: 0.1u, Capacitor_THT:C_Disc_D3.0mm_W2.0mm_P2.50mm, symbol PCM_SL_Devices:Capacitor_NP
- added C3, C5: 10u, symbol Device:C_Polarized
- added C6: 1u, Capacitor_THT:C_Disc_D3.0mm_W2.0mm_P2.50mm, symbol PCM_SL_Devices:Capacitor_NP
- added F1: 0ZCH0110AF2E, FUSC3226X100N, symbol 0ZCH0110AF2E:0ZCH0110AF2E
- added J1: SS-52400-002, SS-52400-002:BELFUSE_SS-52400-002, symbol SS-52400-002:SS-52400-002
- added J2: B2B-PH-SM4-TB, B2B-PH-SM4-TB:JST_B2B-PH-SM4-TB, symbol B2B-PH-SM4-TB:B2B-PH-SM4-TB
- added LED1: LTST-C170TBKT, LEDC2012X120N, symbol LTST-C170TBKT:LTST-C170TBKT
- added LED2: LTST-C170GKT, LEDC2012X120N, symbol LTST-C170GKT:LTST-C170GKT
- added LED4, LED5: LTST-C170KRKT, LEDC2012X120N, symbol LTST-C170KRKT:LTST-C170KRKT
- added R1, R2: 10K, symbol Device:R
- added R10, R7, R8, R9: 470, symbol Device:R
- added R3, R4: 5.1K, symbol Device:R
- added R5: 2K, symbol Device:R
- added R6: 20K, symbol Device:R
- added U1: MCP73871-2CAI_ML, MCP73871-2CAI_ML:QFN50P400X400X100-21N, symbol MCP73871-2CAI_ML:MCP73871-2CAI_ML
- added VR1: LM1117MPX-3.3, LM1117MPX-3.3:VREG_LM1117MPX-3.3, symbol LM1117MPX-3.3:LM1117MPX-3.3
Connections:
- new net: R9.2, U1.6 (~{PG})
- new net: R6.1, U1.12 (PROG3)
- new net: R8.2, U1.8 (STAT1/~{LBO})
- new net: R5.2, U1.13 (PROG1)
- new net: R2.2, U1.5 (THERM)
- new net: R7.1, U1.7 (STAT2)
- new net: R1.1, U1.9 (~{TE})
- new net: J1.A5 (CC1), R4.1
- new net: J1.B5 (CC2), R3.1
- new net: LED4.1 (K), R10.1
- new net +5V_USB: C6.2, F1.2, LED1.2 (A), LED2.2 (A), LED5.2 (A), U1.17 (CE), U1.18 (IN), U1.19 (IN), U1.2 (VPCC), U1.4 (PROG2)
- new net 3.3V: C4.2, C5.1, LED4.2 (A), VR1.2 (VOUT_2), VR1.4 (VOUT_4)
- new net 5V: C2.2, C3.1, U1.1 (OUT), U1.20 (OUT), VR1.3 (VIN)
- new net CHARGED: LED2.1 (K), R8.1
- new net CHARGING: LED5.1 (K), R9.1
- new net CHARGING_POWER_GOOD: LED1.1 (K), R7.2
- new net GND: C1.1, C2.1, C3.2, C4.1, C5.2, C6.1, J1.A1 (GNDA1), J1.A12 (GNDA2), J1.B1 (GNDB1), J1.B12 (GNDB2), J1.G1 (GND/SHIELD), J1.G2 (GND/SHIELD), J1.G3 (GND/SHIELD), J1.G4 (GND/SHIELD), J1.S1 (GND/SHIELD), J1.S2 (GND/SHIELD), J1.S3 (GND/SHIELD), J1.S4 (GND/SHIELD), J2.1, R1.2, R10.2, R2.1, R3.2, R4.2, R5.1, R6.2, U1.10 (VSS), U1.11 (VSS), U1.21 (VSS), VR1.1 (GND)
- new net USB_DN: J1.A7 (DN1), J1.B7 (DN2)
- new net USB_DP: J1.A6 (DP1), J1.B6 (DP2)
- new net VBAT: J2.2, U1.14 (VBAT), U1.15 (VBAT), U1.16 (VBAT_SENSE)
- new net VBUS: C1.2, F1.1, J1.A4 (VBUSA1), J1.A9 (VBUSA2), J1.B4 (VBUSB1), J1.B9 (VBUSB2)
- no-connect marks 0 -> 10
Other:
- added sheet ESP32-C3-02 (ESP32-C3-02.kicad_sch)
- note added: "Battery JS1 connector"
- note added: "LDO(Low dropout voltage regulator)"
- note added: "Lipo battery charger"
- note added: "Power indicator LED"
- note added: "USB-C Connector"
- company: (none) -> JPIndustries
- title: (none) -> ESP32 Sensor board manager

Commit message: esp32 page and datasheets
Other:
- sheet ESP32-C3-02 ports: added USB_DN, USB_DP, V_BUS; removed none
Changed lines of the file:
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@@
 		)
 	)
+	(label "USB_DN"
+		(at 161.29 109.22 180)
+		(effects
+			(font
+				(size 1.27 1.27)
+			)
+			(justify right bottom)
+		)
+	)
 	(label "VBAT"
 		(at 180.34 72.39 180)
@@
 		)
 	)
+	(label "USB_DP"
+		(at 161.29 111.76 180)
+		(effects
+			(font
+				(size 1.27 1.27)
+			)
+			(justify right bottom)
+		)
+	)
 	(label "CHARGED"
 		(at 242.57 63.5 0)
@@
 		)
 	)
+	(label "VBUS"
+		(at 161.29 114.3 180)
+		(effects
+			(font
+				(size 1.27 1.27)
+			)
+			(justify right bottom)
+		)
+	)
 	(label "USB_DP"
 		(at 74.93 54.61 0)
@@
 			)
 		)
+		(pin "USB_DN" input
+			(at 161.29 109.22 180)
+			(effects
+				(font
+					(size 1.27 1.27)
+				)
+				(justify left)
+			)
+		)
+		(pin "USB_DP" input
+			(at 161.29 111.76 180)
+			(effects
+				(font
+					(size 1.27 1.27)
+				)
+				(justify left)
+			)
+		)
+		(pin "V_BUS" input
+			(at 161.29 114.3 180)
+			(effects
+				(font
+					(size 1.27 1.27)
+				)
+				(justify left)
+			)
+		)

Commit message: sensor and user interface done
Parts:
- C1, C2, C4, C6: footprint Capacitor_THT:C_Disc_D3.0mm_W2.0mm_P2.50mm -> Capacitor_SMD:C_0805_2012Metric
- C3, C5: footprint (none) -> esp32_manager_project:T491A
- F1: footprint FUSC3226X100N -> esp32_manager_project:FUSC3226X100N
- LED1, LED2, LED4: footprint LEDC2012X120N -> esp32_manager_project:LEDC2012X120N
- LED3: renamed from LED5; footprint LEDC2012X120N -> esp32_manager_project:LEDC2012X120N
- R1, R10, R2, R3, R4, R5, R6, R7, R8, R9: footprint (none) -> Resistor_SMD:R_0805_2012Metric
Connections:
- net GND: now also U1.3 (SEL)
- net 5V renamed +5V

Commit message: corrected erc errors
Parts:
- removed LED1: LTST-C170TBKT, esp32_manager_project:LEDC2012X120N, symbol LTST-C170TBKT:LTST-C170TBKT
- removed LED2: LTST-C170GKT, esp32_manager_project:LEDC2012X120N, symbol LTST-C170GKT:LTST-C170GKT
- removed LED3: LTST-C170KRKT, esp32_manager_project:LEDC2012X120N, symbol LTST-C170KRKT:LTST-C170KRKT
- removed R1, R2: 10K, Resistor_SMD:R_0805_2012Metric, symbol Device:R
- removed R5: 2K, Resistor_SMD:R_0805_2012Metric, symbol Device:R
- removed R6: 20K, Resistor_SMD:R_0805_2012Metric, symbol Device:R
- removed U1: MCP73871-2CAI_ML, MCP73871-2CAI_ML:QFN50P400X400X100-21N, symbol MCP73871-2CAI_ML:MCP73871-2CAI_ML
- added LED7: LTST-C170KRKT, esp32_manager_project:LEDC2012X120N, symbol LTST-C170KRKT:LTST-C170KRKT
- added LED8: LTST-C170TBKT, esp32_manager_project:LEDC2012X120N, symbol LTST-C170TBKT:LTST-C170TBKT
- added LED9: LTST-C170GKT, esp32_manager_project:LEDC2012X120N, symbol LTST-C170GKT:LTST-C170GKT
- added R21, R29: 10K, Resistor_SMD:R_0805_2012Metric, symbol Device:R
- added R35: 20K, Resistor_SMD:R_0805_2012Metric, symbol Device:R
- added R36: 2K, Resistor_SMD:R_0805_2012Metric, symbol Device:R
- added U1: MCP73871, Package_DFN_QFN:QFN-20-1EP_4x4mm_P0.5mm_EP2.5x2.5mm, symbol Battery_Management:MCP73871
- C6: footprint Capacitor_SMD:C_0805_2012Metric -> Capacitor_THT:C_Disc_D3.0mm_W2.0mm_P2.50mm
Connections:
- net +5V: now also U1.1 (OUT), U1.20 (OUT)
- net +5V_USB: now also C6.1, LED7.2 (A), LED8.2 (A), LED9.2 (A), U1.17 (CE), U1.18 (IN), U1.19 (IN), U1.2 (VPCC), U1.4 (PROG2); no longer C6.2
- net CHARGED: now also R7.2, LED9.1 (K); no longer R8.1
- net CHARGING: now also LED7.1 (K)
- net CHARGING_POWER_GOOD: now also R8.1, LED8.1 (K); no longer R7.2
- net GND: now also C6.2, R21.2, R29.2, R35.2, R36.1, U1.10 (V_{SS}), U1.11 (V_{SS}), U1.21 (V_{SS}), U1.3 (SEL); no longer C6.1
- net VBAT: now also U1.14 (V_{BAT}), U1.15 (V_{BAT}), U1.16 (V_{BAT_SENSE})
- net at R9.2: now also U1.6 (~{PG})
- net at R8.2: now also U1.7 (STAT2)
- net at R7.1: now also U1.8 (STAT1/~{LBO})
- new net: R35.1, U1.12 (PROG3)
- new net: R36.2, U1.13 (PROG1)
- new net: R29.1, U1.5 (THERM)
- new net: R21.1, U1.9 (~{TE})
Other:
- moved on the sheet: R7, R8, R9

Commit message: finished design of pcb, next copper zones, routing
Parts:
- J1: footprint SS-52400-002:BELFUSE_SS-52400-002 -> esp32_manager_project:BELFUSE_SS-52400-002
- J2: footprint B2B-PH-SM4-TB:JST_B2B-PH-SM4-TB -> esp32_manager_project:JST_B2B-PH-SM4-TB
- VR1: footprint LM1117MPX-3.3:VREG_LM1117MPX-3.3 -> esp32_manager_project:VREG_LM1117MPX-3.3
Changed lines of the file:
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@@
 			)
 		)
-		(property "Footprint" "B2B-PH-SM4-TB:JST_B2B-PH-SM4-TB"
+		(property "Footprint" "esp32_manager_project:JST_B2B-PH-SM4-TB"
 			(at 27.94 160.02 0)
 			(effects
@@
 			)
 		)
-		(property "Footprint" "SS-52400-002:BELFUSE_SS-52400-002"
+		(property "Footprint" "esp32_manager_project:BELFUSE_SS-52400-002"
 			(at 54.61 57.15 0)
 			(effects
@@
 			)
 		)
-		(property "Footprint" "LM1117MPX-3.3:VREG_LM1117MPX-3.3"
+		(property "Footprint" "esp32_manager_project:VREG_LM1117MPX-3.3"
 			(at 60.96 114.3 0)
 			(effects

Commit message: finish esp32
Parts:
- added F2: 0ZCH0110AF2E, FUSC3226X100N, symbol 0ZCH0110AF2E:0ZCH0110AF2E
Connections:
- net +5V: now also F2.2; no longer U1.1 (OUT), U1.20 (OUT)
- new net: F2.1, U1.1 (OUT), U1.20 (OUT)
Changed lines of the file:
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@@
 	(wire
 		(pts
+			(xy 236.22 95.25) (xy 236.22 97.79)
+		)
+		(stroke
+			(width 0)
+			(type default)
+		)
+	)
+	(wire
+		(pts
 			(xy 200.66 77.47) (xy 198.12 77.47)
 		)
@@
 	(symbol
 		(lib_id "power:+5V")
-		(at 236.22 77.47 270)
+		(at 236.22 97.79 270)
 		(unit 1)
 		(exclude_from_sim no)
@@
 		(fields_autoplaced yes)
 		(property "Reference" "#PWR058"
-			(at 232.41 77.47 0)
+			(at 232.41 97.79 0)
 			(effects
 				(font
@@
 		)
 		(property "Value" "+5V"
-			(at 240.03 77.4699 90)
+			(at 240.03 97.7899 90)
 			(effects
 				(font
@@
 		)
 		(property "Footprint" ""
-			(at 236.22 77.47 0)
+			(at 236.22 97.79 0)
 			(effects
 				(font
@@
 		)
 		(property "Datasheet" ""
-			(at 236.22 77.47 0)
+			(at 236.22 97.79 0)
 			(effects
 				(font
@@
 		)
 		(property "Description" "Power symbol creates a global label with name \"+5V\""
-			(at 236.22 77.47 0)
+			(at 236.22 97.79 0)
 			(effects
 				(font
@@
 					(unit 1)
 				)
+			)
+		)
+	)
+	(symbol
+		(lib_id "0ZCH0110AF2E:0ZCH0110AF2E")
+		(at 236.22 77.47 270)
+		(unit 1)
+		(exclude_from_sim no)
+		(in_bom yes)
+		(on_board yes)
+		(dnp no)
+		(fields_autoplaced yes)
+		(property "Reference" "F2"
+			(at 238.76 85.0899 90)
+			(effects
+				(font
+					(size 1.27 1.27)
+				)
+				(justify left)
+			)
+		)
+		(property "Value" "0ZCH0110AF2E"
+			(at 238.76 87.6299 90)
+			(effects
+				(font
+					(size 1.27 1.27)
+				)
+				(justify left)
+			)
+		)
+		(property "Footprint" "FUSC3226X100N"
+			(at 140.03 91.44 0)
+			(effects
+				(font
+					(size 1.27 1.27)
+				)
+				(justify left top)
+				(hide yes)
+			)
+		)
+		(property "Datasheet" "https://www.belfuse.com/resources/datasheets/circuitprotection/ds-cp-0zch-series.pdf"
+			(at 40.03 91.44 0)
+			(effects
+				(font
+					(size 1.27 1.27)
+				)
+				(justify left top)
+				(hide yes)
+			)
+		)
+		(property "Description" "1210 SMT PPTC | 1.10 Ih | 16V"
+			(at 236.22 77.47 0)
+			(effects
+				(font
+					(size 1.27 1.27)
+				)
+				(hide yes)
+			)
+		)
+		(property "Height" "1"
+			(at -159.97 91.44 0)
+			(effects
+				(font
+					(size 1.27 1.27)
+				)
+				(justify left top)
+				(hide yes)
+			)
+		)
+		(property "Manufacturer_Name" "Bel Circuit Protection"
+			(at -259.97 91.44 0)
+			(effects
+				(font
+					(size 1.27 1.27)
+				)
+				(justify left top)
+				(hide yes)
+			)
+		)
+		(property "Manufacturer_Part_Number" "0ZCH0110AF2E"
+			(at -359.97 91.44 0)
+			(effects
+				(font
+					(size 1.27 1.27)
+				)
+				(justify left top)
+				(hide yes)
+			)
+		)
+		(property "Mouser Part Number" ""
+			(at -459.97 91.44 0)
+			(effects
+				(font
+					(size 1.27 1.27)
+				)
+				(justify left top)
+				(hide yes)
+			)
+		)
+		(property "Mouser Price/Stock" ""
+			(at -559.97 91.44 0)
+			(effects
+				(font
+					(size 1.27 1.27)
+				)
+				(justify left top)
+				(hide yes)
+			)
+		)
+		(property "Arrow Part Number" ""
+			(at -659.97 91.44 0)
+			(effects
+				(font
+					(size 1.27 1.27)
+				)
+				(justify left top)
+				(hide yes)
+			)
+		)
+		(property "Arrow Price/Stock" ""
+			(at -759.97 91.44 0)
+			(effects
+				(font
+					(size 1.27 1.27)
+				)
+				(justify left top)
+				(hide yes)
+			)
+		)
+		(pin "2"
+		)
+		(pin "1"
+		)
+		(instances
+			(project ""
+				(path "/6166e74a-1734-44f8-8d71-dfcab5cab94e"
+					(reference "F2")
+					(unit 1)
+				)
